File: KiCad/ChargerTester/ChargerTester.kicad_sch (KiCad schematic)
At the start: 31 parts, among them Q1 IRF2807, SW1 YES, U1 LH1526, U2 LH1526, U3 CPC1030, U4 LM317T, U5 LM317T, U6 LM317T

Commit message: KiCad. fixed 100 ohms on gate
Parts:
- added R?: 100 Ом, symbol Device:R
Connections:
- net load_on_pin D3 (3): now also R?.2; no longer Q1.1 (G)
- new net: Q1.1 (G), R?.1
Changed lines of the file:
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@@
+    (stroke (width 0) (type default) (color 0 0 0 0))
+  )
+  (wire (pts (xy 147.32 139.7) (xy 143.51 139.7))
     (stroke (width 0) (type default) (color 0 0 0 0))
   )
@@
   )
   (polyline (pts (xy 162.56 177.8) (xy 19.05 177.8))
+    (stroke (width 0) (type default) (color 0 0 0 0))
+  )
+  (wire (pts (xy 133.35 139.7) (xy 135.89 139.7))
     (stroke (width 0) (type default) (color 0 0 0 0))
   )
@@
     (effects (font (size 1.27 1.27)) (justify left bottom))
   )
-  (label "load_on_pin D3 (3)" (at 133.35 139.7 0)
+  (label "load_on_pin D3 (3)" (at 147.32 139.7 90)
     (effects (font (size 1.27 1.27)) (justify left bottom))
   )
@@
     (pin "2")
     (pin "3")
+  )
+  (symbol (lib_id "Device:R") (at 139.7 139.7 90) (unit 1)
+    (in_bom yes) (on_board yes) (fields_autoplaced)
+    (property "Reference" "R?" (id 0) (at 139.7 133.35 90))
+    (property "Value" "100 Ом" (id 1) (at 139.7 135.89 90))
+    (property "Footprint" "" (id 2) (at 139.7 141.478 90)
+      (effects (font (size 1.27 1.27)) hide)
+    )
+    (property "Datasheet" "~" (id 3) (at 139.7 139.7 0)
+      (effects (font (size 1.27 1.27)) hide)
+    )
+    (pin "1")
+    (pin "2")
   )
   (symbol (lib_id "Device:R") (at 104.14 62.23 0) (unit 1)
@@
       (reference "R16") (unit 1) (value "2,7 кОм") (footprint "")
     )
+    (path "/7f093f1d-323b-4b4e-b33a-3f6815b22768"
+      (reference "R?") (unit 1) (value "100 Ом") (footprint "")
+    )
     (path "/5fd5bf5a-0e10-459c-b306-5d7f6469d475"
